Commit message: Update ur20

File: robots/ur20/urdf/ur20.urdf (robot description, URDF)
Before this commit: robot ur20_robot, 11 links, 10 joints
Links:
- link base_link_inertia: geometry collision mesh filename=pacakge://ur20/meshes/collision/base.stl; visual mesh filename=pacakge://ur20/meshes/visual/base.dae
- link forearm_link: geometry collision mesh filename=pacakge://ur20/meshes/collision/forearm.stl; visual mesh filename=pacakge://ur20/meshes/visual/forearm.dae
- link shoulder_link: geometry collision mesh filename=pacakge://ur20/meshes/collision/shoulder.stl; visual mesh filename=pacakge://ur20/meshes/visual/shoulder.dae
- link upper_arm_link: geometry collision mesh filename=pacakge://ur20/meshes/collision/upperarm.stl; visual mesh filename=pacakge://ur20/meshes/visual/upperarm.dae
- link wrist_1_link: geometry collision mesh filename=pacakge://ur20/meshes/collision/wrist1.stl; visual mesh filename=pacakge://ur20/meshes/visual/wrist1.dae
- link wrist_2_link: geometry collision mesh filename=pacakge://ur20/meshes/collision/wrist2.stl; visual mesh filename=pacakge://ur20/meshes/visual/wrist2.dae
- link wrist_3_link: geometry collision mesh filename=pacakge://ur20/meshes/collision/wrist3.stl; visual mesh filename=pacakge://ur20/meshes/visual/wrist3.dae

Commit message: update ur20

File: robots/ur20/urdf/ur20.urdf (robot description, URDF)
Before this commit: robot ur20_robot, 11 links, 10 joints
Links:
- link base_link_inertia: geometry collision mesh filename=package://ur20/meshes/collision/base.stl; visual mesh filename=package://ur20/meshes/visual/base.dae
- link forearm_link: geometry collision mesh filename=package://ur20/meshes/collision/forearm.stl; visual mesh filename=package://ur20/meshes/visual/forearm.dae
- link shoulder_link: geometry collision mesh filename=package://ur20/meshes/collision/shoulder.stl; visual mesh filename=package://ur20/meshes/visual/shoulder.dae
- link upper_arm_link: geometry collision mesh filename=package://ur20/meshes/collision/upperarm.stl; visual mesh filename=package://ur20/meshes/visual/upperarm.dae
- link wrist_1_link: geometry collision mesh filename=package://ur20/meshes/collision/wrist1.stl; visual mesh filename=package://ur20/meshes/visual/wrist1.dae
- link wrist_2_link: geometry collision mesh filename=package://ur20/meshes/collision/wrist2.stl; visual mesh filename=package://ur20/meshes/visual/wrist2.dae
- link wrist_3_link: geometry collision mesh filename=package://ur20/meshes/collision/wrist3.stl; visual mesh filename=package://ur20/meshes/visual/wrist3.dae
